Commit message: add imu data to simulation

File: turorial_diff/install/my_robot/share/my_robot/urdf/my_robot.urdf (robot description, URDF)
Before this commit: robot my_robot, 4 links, 3 joints
Links:
- added link imu_link, mass 0.01; collision sphere radius=0.01; visual sphere radius=0.01
Joints:
- added joint imu_joint: type fixed, parent base_link, child imu_link
